File: free2breathe_pcb/free2breathe_pcb.kicad_sch (KiCad schematic)
At the start: 66 parts, among them J1 LED_Connector, J2 Alarm_Connector, J3 LED_Power, P1 USB_C_Plug_USB2.0, Q1 DMN3404L, Q2 AO3401A, SW1 SW_SPST, U1 IP5328, U2 CO Sensor, U3 O3 Sensor, U4 NO2 Sensor, U5 SO2 Sensor

Commit message: add sensor biasing, assign footprints
Parts:
- removed J1: LED_Connector, Connector_JST:JST_PH_B2B-PH-K_1x02_P2.00mm_Vertical, symbol Connector:Conn_01x02_Female
- removed J3: LED_Power, symbol Connector:Conn_01x02_Female
- removed P1: USB_C_Plug_USB2.0, symbol Connector:USB_C_Plug_USB2.0
- removed U3: O3 Sensor, components:XDCR_110-102, symbol 110-102:110-102
- removed U4: NO2 Sensor, components:XDCR_110-102, symbol 110-102:110-102
- added BT1, BT2: Battery_Cell, switch:switch_pad, symbol Device:Battery_Cell
- added C18, C19, C20, C21, C22, C23, C24, C25, C26, C27, C28, C29, C30, C31, C32, C33: 0.1u, Capacitor_SMD:C_0603_1608Metric, symbol Device:C
- added J1: LED_Connector, Connector_JST:JST_PH_B3B-PH-K_1x03_P2.00mm_Vertical, symbol Connector:Conn_01x03_Female
- added R25, R26, R27, R34, R35, R36, R37, R38, R39, R40, R41, R42, R43: 10, Resistor_SMD:R_0603_1608Metric, symbol Device:R
- added R28, R31: 10k, Resistor_SMD:R_0603_1608Metric, symbol Device:R
- added R29, R32: 910, Resistor_SMD:R_0603_1608Metric, symbol Device:R
- added R30, R33: 4.7k, Resistor_SMD:R_0603_1608Metric, symbol Device:R
- added U3, U4, U6, U7: MCP6044-E/P, components:DIP254P762X533-14, symbol MCP6044-E_P:MCP6044-E/P
- added U8: O3 Sensor, components:XDCR_110-102, symbol 110-102:110-102
- added U9: NO2 Sensor, components:XDCR_110-102, symbol 110-102:110-102
- BT3: footprint (none) -> switch:switch_pad
- D1, D2, D3, D4, D5, D6, D7, D8, D9: footprint (none) -> LED_SMD:LED_0805_2012Metric
- L1: footprint (none) -> components:IND_AMPLA5030S2R2MT
- R10: value 10k -> 910
- R11: value 100k -> 10k
- R13, R2: value 100k -> 4.7k
- R14, R16, R17, R18, R19, R20: value 10k -> 10
- R15: value 100k -> 10
- R21, R22, R23, R24: footprint (none) -> Resistor_SMD:R_0603_1608Metric
- SW1: value SW_SPST -> Power_Switch
- TH1: footprint (none) -> Resistor_SMD:R_0805_2012Metric
- U1: footprint (none) -> Package_DFN_QFN:QFN-40-1EP_6x6mm_P0.5mm_EP4.6x4.6mm
Connections:
- net Arduino_3V3: now also R11.2, R12.1, R28.1, R31.1, U3.4 (VDD), U4.4 (VDD), U6.4 (VDD), U7.4 (VDD); no longer R11.1, R13.1, R15.1, R2.1
- net Arduino_5V: now also J1.1 (Pin_1)
- net Arduino_A0: no longer R17.2, U2.4 (REFERENCE), U2.5 (COUNTER)
- net Arduino_A1: no longer R10.1, R17.1, R2.2, U2.1 (WORKING), U2.6 (WORKING)
- net Arduino_A2: no longer R18.1
- net Arduino_A3: no longer R11.2, R12.1, R18.2
- net Arduino_A4: no longer R19.1
- net Arduino_A5: no longer R13.2, R14.1, R19.2
- net Arduino_A6: no longer R20.1, U5.4 (REFERENCE), U5.5 (COUNTER)
- net Arduino_A7: no longer R15.2, R16.1, R20.2, U5.1 (WORKING), U5.6 (WORKING)
- net Arduino_D8: now also J1.2 (Pin_2)
- net GND: now also R13.2, R2.1, BT1.2 (-), BT2.2 (-), C18.2, C19.2, C20.2, C21.2, C26.2, C27.2, C28.2, C29.2, J1.3 (Pin_3), R30.2, R33.2, U3.11 (VSS), U4.11 (VSS), U6.11 (VSS), U7.11 (VSS); no longer R10.2, R12.2, R14.2, R16.2
- net at BT3.1 (+), SW1.1 (A): now also BT1.1 (+), BT2.1 (+)
- new net: C32.1, R42.1, U6.1 (VOUTA)
- new net: C32.2, U6.2 (VINA-), U8.4 (REFERENCE)
- new net: C31.1, R39.2, U7.12 (VIND+), U7.7 (VOUTB)
- new net: C31.2, R39.1, R41.2, U7.10 (VINC+), U7.6 (VINB-)
- new net: C28.1, R36.2, U7.3 (VINA+)
- new net: C22.2, R18.1, R20.2, U3.10 (VINC+), U3.6 (VINB-)
- new net: C22.1, R18.2, U3.12 (VIND+), U3.7 (VOUTB)
- new net: C24.1, R26.1, U3.1 (VOUTA)
- new net: C24.2, U2.4 (REFERENCE), U3.2 (VINA-)
- new net: C18.1, R14.2, U3.3 (VINA+)
- new net: C19.1, R15.2, U3.5 (VINB+)
- new net: C23.2, R19.1, R25.2, U4.10 (VINC+), U4.6 (VINB-)
- new net: C23.1, R19.2, U4.12 (VIND+), U4.7 (VOUTB)
- new net: R41.1, U9.1 (WORKING), U9.6 (WORKING)
- new net: C25.1, R27.1, U4.1 (VOUTA)
- new net: R27.2, U5.5 (COUNTER)
- new net: R28.2, R29.1, R34.1
- new net: R29.2, R30.1, R35.1
- new net: C33.1, R43.1, U7.1 (VOUTA)
- new net: C33.2, U7.2 (VINA-), U9.4 (REFERENCE)
- new net: C29.1, R37.2, U7.5 (VINB+)
- new net: R31.2, R32.1, R36.1
- new net: R32.2, R33.1, R37.1
- new net: C30.2, R38.1, R40.2, U6.10 (VINC+), U6.6 (VINB-)
- new net: C30.1, R38.2, U6.12 (VIND+), U6.7 (VOUTB)
- new net: C26.1, R34.2, U6.3 (VINA+)
- new net: R40.1, U8.1 (WORKING), U8.6 (WORKING)
- new net: C25.2, U4.2 (VINA-), U5.4 (REFERENCE)
- new net: R43.2, U9.5 (COUNTER)
- new net: R10.1, R16.1, R2.2
- new net: C20.1, R16.2, U4.3 (VINA+)
- new net: R42.2, U8.5 (COUNTER)
- new net: R20.1, U2.1 (WORKING), U2.6 (WORKING)
- new net: R10.2, R11.1, R17.1
- new net: C21.1, R17.2, U4.5 (VINB+)
- new net: R26.2, U2.5 (COUNTER)
- new net: R25.1, U5.1 (WORKING), U5.6 (WORKING)
- new net: C27.1, R35.2, U6.5 (VINB+)
- new net 1.024V: R12.2, R13.1, R14.1, R15.1
- new net CO_TP1: U3.13 (VIND-), U3.14 (VOUTD)
- new net CO_TP2: U3.8 (VOUTC), U3.9 (VINC-)
- new net NO2_TP1: U7.13 (VIND-), U7.14 (VOUTD)
- new net NO2_TP2: U7.8 (VOUTC), U7.9 (VINC-)
- new net O3_TP1: U6.13 (VIND-), U6.14 (VOUTD)
- new net O3_TP2: U6.8 (VOUTC), U6.9 (VINC-)
- new net SO2_TP1: U4.13 (VIND-), U4.14 (VOUTD)
- new net SO2_TP2: U4.8 (VOUTC), U4.9 (VINC-)
Other:
- note added: "CO: 0mV"
- note added: "NO2: -200mV"
- note added: "O3: -200mV"
- note added: "SO2: +200mV"
- moved on the sheet: BT3, C2, Q2, R1, SW1, U2

Commit message: additional footprints, update todo
Parts:
- removed C19: 0.1u, Capacitor_SMD:C_0603_1608Metric, symbol Device:C
- removed R15: 10, Resistor_SMD:R_0603_1608Metric, symbol Device:R
- removed R28, R31: 10k, Resistor_SMD:R_0603_1608Metric, symbol Device:R
- removed R29, R32: 910, Resistor_SMD:R_0603_1608Metric, symbol Device:R
- removed R30, R33: 4.7k, Resistor_SMD:R_0603_1608Metric, symbol Device:R
- R11: value 10k -> 4.7k
- R2: value 4.7k -> 10k
Connections:
- net Arduino_3V3: now also R2.1; no longer R11.2
- net GND: now also R11.2; no longer R2.1
- net at C18.1, R14.2, U3.3 (VINA+): now also U3.5 (VINB+)
- net Divider_High: now reaches R34.1
- net Divider_High: now also R10.1, R17.1, R2.2, R36.1
- net Divider_Low: now reaches R35.1
- net Divider_Low: now also R10.2, R11.1, R16.1, R37.1
Other:
- moved on the sheet: C18, C20, C21, C22, C23, C24, C25, C26, C27, C28, C29, C30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

Commit message: completed rev1 board schematic
Parts:
- removed C16: 220uF 25V, Capacitor_SMD:C_0201_0603Metric, symbol Device:C_Polarized
- removed D1, D2, D3, D4: LED, LED_SMD:LED_0805_2012Metric, symbol Device:LED
- added C16: 10uF 25V, Capacitor_SMD:C_0603_1608Metric, symbol Device:C
- added D6, D7, D8, D9: LED, LED_SMD:LED_0603_1608Metric, symbol Device:LED
- added J3: USB4110-GF-A_REVB, components:GCT_USB4110-GF-A_REVB, symbol USB4110-GF-A_REVB:USB4110-GF-A_REVB
- C1, C10, C11, C12, C13, C14, C15, C17, C2, C3, C4, C5, C6, C7, C8: footprint Capacitor_SMD:C_0201_0603Metric -> Capacitor_SMD:C_0603_1608Metric
- C9: value NC/22uF 25V -> 22uF 25V; footprint Capacitor_SMD:C_0201_0603Metric -> Capacitor_SMD:C_0603_1608Metric
- D1: renamed from D6; footprint LED_SMD:LED_0805_2012Metric -> LED_THT:LED_D4.0mm
- D2: renamed from D7; footprint LED_SMD:LED_0805_2012Metric -> LED_THT:LED_D4.0mm
- D3: renamed from D8; footprint LED_SMD:LED_0805_2012Metric -> LED_THT:LED_D4.0mm
- D4: renamed from D9; footprint LED_SMD:LED_0805_2012Metric -> LED_THT:LED_D4.0mm
- D5: footprint LED_SMD:LED_0805_2012Metric -> LED_SMD:LED_0603_1608Metric
- R3: value 0.01 -> 10m
- renumbered U3 to U2, U2 to U3, U8 to U7, U7 to U8
Connections:
- net CO_TP1 is gone; now on net Arduino_A0: U2.13 (VIND-), U2.14 (VOUTD)
- net CO_TP2 is gone; now on net Arduino_A1: U2.8 (VOUTC), U2.9 (VINC-)
- net NO2_TP1 is gone; now on net Arduino_A6: U8.13 (VIND-), U8.14 (VOUTD)
- net NO2_TP2 is gone; now on net Arduino_A7: U8.8 (VOUTC), U8.9 (VINC-)
- net O3_TP1 is gone; now on net Arduino_A4: U6.13 (VIND-), U6.14 (VOUTD)
- net O3_TP2 is gone; now on net Arduino_A5: U6.8 (VOUTC), U6.9 (VINC-)
- net SO2_TP1 is gone; now on net Arduino_A2: U4.13 (VIND-), U4.14 (VOUTD)
- net SO2_TP2 is gone; now on net Arduino_A3: U4.8 (VOUTC), U4.9 (VINC-)
- net CC1: now also J3.A5 (CC1)
- net CC2: now also J3.B5 (CC2)
- net DMC: now also J3.A7 (DN1)
- net DPC: now also J3.A6 (DP1)
- net GND: now also C16.2, D9.1 (K), J3.A1/B12 (GND), J3.B1/A12 (GND), J3.S1 (GND), J3.S2 (GND), J3.S3 (GND), J3.S4 (GND)
- net VBAT+: now also BT1.1 (+), BT2.1 (+), BT3.1 (+), C3.2, U1.28 (BAT); no longer SW1.2 (B)
- net VBUS: now also J3.A4/B9 (VBUS), J3.B4/A9 (VBUS)
- net VSYS: now also C16.1
- net at D5.1 (K): now also R9.1, U1.13 (L3), D6.2 (A), D7.1 (K), D8.2 (A); no longer R7.2
- net at U1.11 (L1): now also R6.1; no longer R7.1
- net at R8.1: now also U1.20 (LIGHT); no longer U1.12 (L2)
- net at R8.2: now also D9.2 (A)
- net at R6.2: now also D5.2 (A), D6.1 (K)
- net DMA1: no longer names the net of U1.38 (DMA1)
- net DMA2: no longer names the net of U1.40 (DMA2)
- net DMB: no longer names the net of U1.6 (DMB)
- net DPA1: no longer names the net of U1.39 (DPA1)
- net DPA2: no longer names the net of U1.1 (DPA2)
- net DPB: no longer names the net of U1.7 (DPB)
- net VIN: no longer names the net of U1.30 (VIN)
- net VING: no longer names the net of U1.31 (VING)
- net VOUT1 renamed VOUT
- net VOUT: now also SW1.1 (A); no longer U1.37 (VOUT1)
- net VOUT1G renamed VOUTG
- net VOUT2: no longer names the net of U1.34 (VOUT2)
- net VOUT2G: no longer names the net of U1.35 (VOUT2G)
- new net: D7.2 (A), D8.1 (K), R7.2
- new net: R7.1, U1.12 (L2)
- new net: SW1.2 (B), U1.37 (VOUT1)
- no-connect marks 3 -> 26
Other:
- note added: "CO_TP1"
- note added: "CO_TP2"
- note added: "NO2_TP1"
- note added: "NO2_TP2"
- note added: "O3_TP1"
- note added: "O3_TP2"
- note added: "SO2_TP1"
- note added: "SO2_TP2"
- moved on the sheet: A1, BT1, BT2, BT3, C1, C10, C11, C12, C13, C14, C15, C17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

Commit message: group sensors with supporting hardware
Parts:
- removed D9: LED, LED_SMD:LED_0603_1608Metric, symbol Device:LED
- removed R8: 100, Resistor_SMD:R_0603_1608Metric, symbol Device:R
- D1, D2, D3, D4: footprint LED_THT:LED_D4.0mm -> LED_THT:LED_D3.0mm
- D5: renamed from D7; footprint LED_SMD:LED_0603_1608Metric -> LED_THT:LED_D3.0mm
- D6: renamed from D8; footprint LED_SMD:LED_0603_1608Metric -> LED_THT:LED_D3.0mm
- D7: renamed from D5; footprint LED_SMD:LED_0603_1608Metric -> LED_THT:LED_D3.0mm
- D8: renamed from D6; footprint LED_SMD:LED_0603_1608Metric -> LED_THT:LED_D3.0mm
- renumbered C2 to C1, C14 to C10, C16 to C11, C8 to C12, C1 to C13, C11 to C14, C13 to C15, C15 to C16, C25 to C18, C24 to C19, C5 to C2, C18 to C21, C23 to C22, C22 to C23, C21 to C24, C32 to C25, C33 to C27, C30 to C29, C6 to C3, C27 to C30, C29 to C32, C3 to C4, C4 to C5, C7 to C6, C9 to C7, C10 to C8, C12 to C9, J3 to J1, J1 to J2, J2 to J3, Q2 to Q1, Q1 to Q2, R9 to R10, R4 to R11, R27 to R12, R12 to R13, R26 to R14, R16 to R15, R14 to R16, R13 to R17, R25 to R18, R20 to R19, R3 to R2, R19 to R20, R18 to R21, R17 to R22, R2 to R23, R10 to R24, R11 to R25, R42 to R26, R43 to R27, R34 to R28, R36 to R29, R5 to R3, R40 to R30, R41 to R31, R38 to R32, R35 to R33, R39 to R34, R37 to R35, R21 to R4, R22 to R5, R23 to R6, R24 to R8, R6 to R9, U4 to U2, U2 to U3, U5 to U4, U3 to U5
Connections:
- no-connect marks 26 -> 27
